File: Receiver/main_design2.sch (EAGLE design)
At the start: 34 parts, among them IC1 7805TV

Commit message: recently printed version, transfer to test on windows mplab
Parts:
- removed C10, C9: 1uf, UMK105CBJ105KV-F:UMK105CBJ105KV-F
- removed R2: 2kR, rcl:R-US_0204/7
- removed U$2: MCP73831, MCP73831:MCP73831
- removed VBAT-IN: .1uf, EMF105B7104MVHF:EMF105B7104MVHF
- added C13: (no value), rcl:C-USC0805
- added C14, C8: 10uf, rcl:C-USC0805
- added C15: 0.1uf, rcl:C-USC0805
- added GND, GND7, GND9, SW1, SW2: (no value), wirepad:1,6/0,8
- added IC2: MCP73831, MCP73831-SOP:MCP73831
- added R3: 2kR, rcl:R-US_0204/7
- added VCC: VCC, wirepad:1,6/0,8
- C1, C7: value .1uf -> 10uf; device EMF105B7104MVHF:EMF105B7104MVHF -> rcl:C-USC0805
- C2: value 1uf -> 0.1uf; device UMK105CBJ105KV-F:UMK105CBJ105KV-F -> rcl:C-USC0805
- C3: value 1uf -> 100uF; device UMK105CBJ105KV-F:UMK105CBJ105KV-F -> rcl:CPOL-USE5-5
- C5: value 330uf -> 100uF; device rcl:CPOL-USE5-10.5 -> rcl:CPOL-USE5-6
- L1: value 2.2uH -> LPS4012-SMD; device rcl:R-US_R0603 -> LPS4012:LPS4012-SMD
Connections:
- removed net N$11: L1.1, U$4.L2
- removed net N$5: R2.2, U$2.PROG
- new net N$21: L1.1, U$4.L1
- new net N$22: L1.2, U$4.L2
- new net PRE-BATIN: 18650+.P, C13.1, IC2.VBAT, SW1.P
- net GND: now also C13.2, C14.2, C15.2, C2.2, C3.-, C7.2, C8.2, GND.P, GND7.P, GND9.P, IC2.VSS, R3.1; no longer C10.1, C2.1, C3.1, C7.1, C9.1, R2.1, U$2.VSS, U$4.PGND@3, VBAT-IN.1
- net N$10: now also IC2.PROG, R3.2; no longer L1.2, U$4.L1
- net N$2: now also C2.1
- net SOL_IN: now also C5.+
- net VBAT-IN: now also C1.2, SW2.P; no longer 18650+.P, C2.2, C9.2, U$2.VBAT@3, U$2.VBAT@4, VBAT-IN.2
- net VIN-5V: now also C14.1, C15.1, IC2.VDD; no longer C1.2, C3.2, U$2.VDD@1, U$2.VDD@2
- net VOUT: now also C3.+, C7.1, C8.1, VCC.P; no longer C10.2, C5.+, C7.2
Other:
- moved on the sheet: C1, C2, C5, C7
