File: Receiver/power.sch (EAGLE design)
At the start: 22 parts, among them IC1 7805TV

Commit message: recently printed version, transfer to test on windows mplab
Parts:
- removed 18650_GND, PAD1: (no value), wirepad:1,6/0,8
- added ANT, DIO0, DIO1, DIO2, DIO3, DIO4, DIO5, GND, GND7, RA4, RA5, RC4, RC5: (no value), wirepad:1,6/0,8
- added C2: 1uf, UMK105CBJ105KV-F:UMK105CBJ105KV-F
- added C4: (no value), rcl:C-USC0402
- added U$5: SRP0510-2R2K, SRP0510-2R2K :SRP0510-2R2K
- C5: value .33uf -> 330uf; device rcl:C-US025-024X044 -> rcl:CPOL-USE5-10.5
- R1: device rcl:R-US_0204/7 -> rcl:R-US_R0805
- U$3: value RFM69C -> RFM69HCW; device RFM69C:RFM69C -> RFM69C:RFM69HCW
Connections:
- net MISO renamed N$1
- removed net N$1 (its old number): C5.1, IC1.VI, SOL_+.P
- new net N$15: DIO1.P, U$3.DIO1
- new net N$16: DIO0.P, U$3.DIO0
- new net N$17: DIO4.P, U$3.DIO4
- new net N$18: DIO3.P, U$3.DIO3
- new net N$19: ANT.P, U$3.ANT
- new net N$20: DIO5.P, U$3.DIO5
- new net N$21: U$4.L1, U$5.1
- new net N$22: U$4.L2, U$5.2
- new net N$3: RA4.P, U$1.RA4
- new net N$6: RA5.P, U$1.RA5
- new net N$7: RC5.P, U$1.RC5
- new net N$8: RC4.P, U$1.RC4
- new net N$9: DIO2.P, U$3.DIO2
- new net SOL_IN: C4.1, IC1.VI, SOL_+.P
- net GND: now also C2.1, C4.2, C5.-, GND.P, GND7.P, U$3.GND; no longer 18650_GND.P, C5.2, U$3.GND@3
- net N$2: now also R1.1; no longer R1.2
- net N$4: now also U$1.RC2, U$3.RESET; no longer PAD1.P, U$3.ANA
- net VBAT-IN: now also C2.2, R1.2; no longer R1.1
- net VOUT: now also C5.+
Other:
- moved on the sheet: R1
